File: stlink.kicad_sch (KiCad schematic)
At the start: 0 parts

Commit message: Update schematic for DebugBoard with connector and power symbols.
Parts:
- added J601: USB_A, Connector_USB:USB_A_Molex_67643_Horizontal, symbol Connector:USB_A
Connections:
- new net +5V: J601.1 (VBUS)
- new net GND: J601.4 (GND), J601.5 (Shield)
- new net USB+: J601.3 (D+)
- new net USB-: J601.2 (D-)

Commit message: Update USB-C and USB-Hub Schematics with New Titles and Reference Changes
- Changed title from "DebugBoard" to "USB-C" in usb_c.kicad_sch.
- Changed title from "DebugBoard" to "USB-Hub" in usb_hub.kicad_sch.
- Updated multiple component references in usb_c.kicad_sch to new identifiers (#PWR0301 to #PWR0312, D301, U301, etc.).
- Updated component reference from "R103" to "R501" in usb_hub.kicad_sch.
Other:
- title: DebugBoard -> ST-Link Interface
Changed lines of the file:
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@@
 	(paper "A4")
 	(title_block
-		(title "DebugBoard")
+		(title "ST-Link Interface")
 		(rev "<<HASH>>")
 		(company "Amateurfunkclub für Remote Stationen")
