File: power.kicad_sch (KiCad schematic)
At the start: 5 parts, among them U104 TLV73333PQDBVRQ1

Commit message: Update USB-C and USB-Hub Schematics with New Titles and Reference Changes
- Changed title from "DebugBoard" to "USB-C" in usb_c.kicad_sch.
- Changed title from "DebugBoard" to "USB-Hub" in usb_hub.kicad_sch.
- Updated multiple component references in usb_c.kicad_sch to new identifiers (#PWR0301 to #PWR0312, D301, U301, etc.).
- Updated component reference from "R103" to "R501" in usb_hub.kicad_sch.
Parts:
- renumbered C111 to C401, C112 to C402, C113 to C403, C115 to C404, U104 to U401
Other:
- title: DebugBoard -> 3V3 Power
Changed lines of the file:
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@@
 	(paper "A4")
 	(title_block
-		(title "DebugBoard")
+		(title "3V3 Power")
 		(rev "<<HASH>>")
 		(company "Amateurfunkclub für Remote Stationen")
@@
 		(dnp no)
 		(fields_autoplaced yes)
-		(property "Reference" "C111"
+		(property "Reference" "C401"
 			(at 121.92 90.1699 0)
 			(effects
@@
 			(project "main"
 				(path "/f228839c-6576-40b2-ae70-679b7b460639/1b089934-e74e-41e6-aad9-3661a2475aec"
-					(reference "C111")
+					(reference "C401")
 					(unit 1)
 				)
@@
 		(dnp no)
 		(fields_autoplaced yes)
-		(property "Reference" "#PWR0126"
+		(property "Reference" "#PWR0402"
 			(at 118.11 104.14 0)
 			(effects
@@
 			(project "main"
 				(path "/f228839c-6576-40b2-ae70-679b7b460639/1b089934-e74e-41e6-aad9-3661a2475aec"
-					(reference "#PWR0126")
+					(reference "#PWR0402")
 					(unit 1)
 				)
@@
 		(dnp no)
 		(fields_autoplaced yes)
-		(property "Reference" "#PWR0140"
+		(property "Reference" "#PWR0407"
 			(at 175.26 104.14 0)
 			(effects
@@
 			(project "main"
 				(path "/f228839c-6576-40b2-ae70-679b7b460639/1b089934-e74e-41e6-aad9-3661a2475aec"
-					(reference "#PWR0140")
+					(reference "#PWR0407")
 					(unit 1)
 				)
@@
 		(dnp no)
 		(fields_autoplaced yes)
-		(property "Reference" "#PWR0131"
+		(property "Reference" "#PWR0404"
 			(at 148.59 102.87 0)
 			(effects
@@
 			(project "main"
 				(path "/f228839c-6576-40b2-ae70-679b7b460639/1b089934-e74e-41e6-aad9-3661a2475aec"
-					(reference "#PWR0131")
+					(reference "#PWR0404")
 					(unit 1)
 				)
@@
 		(dnp no)
 		(fields_autoplaced yes)
-		(property "Reference" "C112"
+		(property "Reference" "C402"
 			(at 135.89 90.1699 0)
 			(effects
@@
 			(project "main"
 				(path "/f228839c-6576-40b2-ae70-679b7b460639/1b089934-e74e-41e6-aad9-3661a2475aec"
-					(reference "C112")
+					(reference "C402")
 					(unit 1)
 				)
@@
 		(dnp no)
 		(fields_autoplaced yes)
-		(property "Reference" "#PWR0139"
+		(property "Reference" "#PWR0406"
 			(at 175.26 85.09 0)
 			(effects
@@
 			(project "main"
 				(path "/f228839c-6576-40b2-ae70-679b7b460639/1b089934-e74e-41e6-aad9-3661a2475aec"
-					(reference "#PWR0139")
+					(reference "#PWR0406")
 					(unit 1)
 				)
@@
 		(dnp no)
 		(fields_autoplaced yes)
-		(property "Reference" "#PWR0129"
+		(property "Reference" "#PWR0403"
 			(at 132.08 104.14 0)
 			(effects
@@
 			(project "main"
 				(path "/f228839c-6576-40b2-ae70-679b7b460639/1b089934-e74e-41e6-aad9-3661a2475aec"
-					(reference "#PWR0129")
+					(reference "#PWR0403")
 					(unit 1)
 				)
@@
 		(dnp no)
 		(fields_autoplaced yes)
-		(property "Reference" "#PWR0135"
+		(property "Reference" "#PWR0405"
 			(at 161.29 104.14 0)
 			(effects
@@
 			(project "main"
 				(path "/f228839c-6576-40b2-ae70-679b7b460639/1b089934-e74e-41e6-aad9-3661a2475aec"
-					(reference "#PWR0135")
+					(reference "#PWR0405")
 					(unit 1)
 				)
@@
 		(dnp no)
 		(fields_autoplaced yes)
-		(property "Reference" "#PWR0125"
+		(property "Reference" "#PWR0401"
 			(at 118.11 85.09 0)
 			(effects
@@
 			(project "main"
 				(path "/f228839c-6576-40b2-ae70-679b7b460639/1b089934-e74e-41e6-aad9-3661a2475aec"
-					(reference "#PWR0125")
+					(reference "#PWR0401")
 					(unit 1)
 				)
@@
 		(dnp no)
 		(fields_autoplaced yes)
-		(property "Reference" "U104"
+		(property "Reference" "U401"
 			(at 148.59 77.47 0)
 			(effects
@@
 			(project "main"
 				(path "/f228839c-6576-40b2-ae70-679b7b460639/1b089934-e74e-41e6-aad9-3661a2475aec"
-					(reference "U104")
+					(reference "U401")
 					(unit 1)
 				)
@@
 		(dnp no)
 		(fields_autoplaced yes)
-		(property "Reference" "C113"
+		(property "Reference" "C403"
 			(at 165.1 88.8999 0)
 			(effects
@@
 			(project "main"
 				(path "/f228839c-6576-40b2-ae70-679b7b460639/1b089934-e74e-41e6-aad9-3661a2475aec"
-					(reference "C113")
+					(reference "C403")
 					(unit 1)
 				)
@@
 		(dnp no)
 		(fields_autoplaced yes)
-		(property "Reference" "C115"
+		(property "Reference" "C404"
 			(at 179.07 88.8999 0)
 			(effects
@@
 			(project "main"
 				(path "/f228839c-6576-40b2-ae70-679b7b460639/1b089934-e74e-41e6-aad9-3661a2475aec"
-					(reference "C115")
-					(unit 1)
-				)
+					(reference "C404")
+					(unit 1)
+				)

Commit message: Refactor code structure for improved readability and maintainability
Connections:
- no-connect marks 2 -> 0
Changed lines of the file:
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@@
 		(color 0 0 0 0)
 	)
-	(no_connect
-		(at 149.86 100.33)
-	)
-	(no_connect
-		(at 149.86 97.79)
-	)
 	(wire
 		(pts
@@
 	(wire
 		(pts
-			(xy 175.26 83.82) (xy 184.15 83.82)
-		)
-		(stroke
-			(width 0)
-			(type default)
-		)
-	)
-	(wire
-		(pts
 			(xy 132.08 86.36) (xy 132.08 87.63)
 		)
@@
 		(pts
 			(xy 175.26 83.82) (xy 175.26 81.28)
-		)
-		(stroke
-			(width 0)
-			(type default)
-		)
-	)
-	(wire
-		(pts
-			(xy 184.15 81.28) (xy 184.15 83.82)
 		)
 		(stroke
@@
 					(unit 1)
 				)
-			)
-		)
-	)
-	(symbol
-		(lib_id "power:PWR_FLAG")
-		(at 184.15 81.28 0)
-		(unit 1)
-		(exclude_from_sim no)
-		(in_bom yes)
-		(on_board yes)
-		(dnp no)
-		(fields_autoplaced yes)
-		(property "Reference" "#FLG0401"
-			(at 184.15 79.375 0)
-			(effects
-				(font
-					(size 1.27 1.27)
-				)
-				(hide yes)
-			)
-		)
-		(property "Value" "PWR_FLAG"
-			(at 184.15 76.2 0)
-			(effects
-				(font
-					(size 1.27 1.27)
-				)
-			)
-		)
-		(property "Footprint" ""
-			(at 184.15 81.28 0)
-			(effects
-				(font
-					(size 1.27 1.27)
-				)
-				(hide yes)
-			)
-		)
-		(property "Datasheet" "~"
-			(at 184.15 81.28 0)
-			(effects
-				(font
-					(size 1.27 1.27)
-				)
-				(hide yes)
-			)
-		)
-		(property "Description" "Special symbol for telling ERC where power comes from"
-			(at 184.15 81.28 0)
-			(effects
-				(font
-					(size 1.27 1.27)
-				)
-				(hide yes)
-			)
-		)
-		(pin "1"
-		)
-		(instances
-			(project "main"
-				(path "/f228839c-6576-40b2-ae70-679b7b460639/1b089934-e74e-41e6-aad9-3661a2475aec"
-					(reference "#FLG0401")
-					(unit 1)
-				)
