File: power_switch.kicad_sch (KiCad schematic)
At the start: 0 parts

Commit message: Update schematic for DebugBoard with connector and power symbols.
Parts:
- added C801: 1uF, Capacitor_SMD:C_0805_2012Metric, symbol Device:C
- added C802: 4.7uF, Capacitor_SMD:C_0805_2012Metric, symbol Device:C
- added U801: TPS22917DBV, Package_TO_SOT_SMD:SOT-23-6, symbol Power_Management:TPS22917DBV
Connections:
- new net +5V: C801.1, U801.1 (VIN)
- new net DUT_VCC: C802.1, U801.5 (QOD), U801.6 (VOUT)
- new net DUT_VCC_EN: U801.3 (ON)
- new net GND: C801.2, C802.2, U801.2 (GND)
- no-connect marks 0 -> 1

Commit message: Update USB-C and USB-Hub Schematics with New Titles and Reference Changes
- Changed title from "DebugBoard" to "USB-C" in usb_c.kicad_sch.
- Changed title from "DebugBoard" to "USB-Hub" in usb_hub.kicad_sch.
- Updated multiple component references in usb_c.kicad_sch to new identifiers (#PWR0301 to #PWR0312, D301, U301, etc.).
- Updated component reference from "R103" to "R501" in usb_hub.kicad_sch.
Other:
- title: DebugBoard -> DUT Power Control
Changed lines of the file:
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@@
 	(paper "A4")
 	(title_block
-		(title "DebugBoard")
+		(title "DUT Power Control")
 		(rev "<<HASH>>")
 		(company "Amateurfunkclub für Remote Stationen")

Commit message: Refactor code structure for improved readability and maintainability
Parts:
- C801: value 1uF -> 4.7u/10V/X5R; MOUSER 791-0805B105K250CT -> 187-CL21A475KAQNNNF
- C802: value 4.7uF -> 4.7u/10V/X5R; MOUSER 791-0805B105K250CT -> 187-CL21A475KAQNNNF
Connections:
- net +5V: now also C801.2; no longer C801.1
- net DUT_VCC: now also C802.2; no longer C802.1, U801.5 (QOD)
- net GND: now also C801.1, C802.1; no longer C801.2, C802.2
- no-connect marks 1 -> 2
