File: ina226.kicad_sch (KiCad schematic)
At the start: 0 parts

Commit message: Update schematic for DebugBoard with connector and power symbols.
Parts:
- added C301: 100n, Capacitor_SMD:C_0805_2012Metric, symbol Device:C
- added R301: 10m, Resistor_SMD:R_2512_6332Metric, symbol Device:R
- added U301: INA226, Package_SO:VSSOP-10_3x3mm_P0.5mm, symbol Sensor_Energy:INA226
Connections:
- new net +5V: C301.1, U301.6 (VS)
- new net A0: U301.2 (A0)
- new net A1: U301.1 (A1)
- new net ALERT: U301.3 (~{Alert})
- new net GND: C301.2, U301.7 (GND)
- new net SCL: U301.5 (SCL)
- new net SDA: U301.4 (SDA)
- new net V_IN: R301.1, U301.10 (Vin+), U301.8 (Vbus)
- new net V_OUT: R301.2, U301.9 (Vin-)

Commit message: Update USB-C and USB-Hub Schematics with New Titles and Reference Changes
- Changed title from "DebugBoard" to "USB-C" in usb_c.kicad_sch.
- Changed title from "DebugBoard" to "USB-Hub" in usb_hub.kicad_sch.
- Updated multiple component references in usb_c.kicad_sch to new identifiers (#PWR0301 to #PWR0312, D301, U301, etc.).
- Updated component reference from "R103" to "R501" in usb_hub.kicad_sch.
Parts:
- renumbered C301 to C901, R301 to R901, U301 to U901
Other:
- title: DebugBoard -> DUT Spannungsmessung
Changed lines of the file:
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@@
 	(paper "A4")
 	(title_block
-		(title "DebugBoard")
+		(title "DUT Spannungsmessung")
 		(rev "<<HASH>>")
 		(company "Amateurfunkclub für Remote Stationen")
@@
 		(dnp no)
 		(fields_autoplaced yes)
-		(property "Reference" "#PWR0301"
+		(property "Reference" "#PWR0902"
 			(at 143.51 107.95 0)
 			(effects
@@
 			(project "main"
 				(path "/f228839c-6576-40b2-ae70-679b7b460639/9647d80f-843f-45c0-950d-b04b6dbce3c2"
-					(reference "#PWR0301")
+					(reference "#PWR0902")
 					(unit 1)
 				)
@@
 		(dnp no)
 		(fields_autoplaced yes)
-		(property "Reference" "C301"
+		(property "Reference" "C901"
 			(at 180.34 81.2799 0)
 			(effects
@@
 			(project "main"
 				(path "/f228839c-6576-40b2-ae70-679b7b460639/9647d80f-843f-45c0-950d-b04b6dbce3c2"
-					(reference "C301")
+					(reference "C901")
 					(unit 1)
 				)
@@
 		(dnp no)
 		(fields_autoplaced yes)
-		(property "Reference" "#PWR0902"
+		(property "Reference" "#PWR0903"
 			(at 176.53 78.74 0)
 			(effects
@@
 			(project "main"
 				(path "/f228839c-6576-40b2-ae70-679b7b460639/9647d80f-843f-45c0-950d-b04b6dbce3c2"
-					(reference "#PWR0902")
+					(reference "#PWR0903")
 					(unit 1)
 				)
@@
 		(dnp no)
 		(fields_autoplaced yes)
-		(property "Reference" "#PWR0302"
+		(property "Reference" "#PWR0904"
 			(at 176.53 95.25 0)
 			(effects
@@
 			(project "main"
 				(path "/f228839c-6576-40b2-ae70-679b7b460639/9647d80f-843f-45c0-950d-b04b6dbce3c2"
-					(reference "#PWR0302")
+					(reference "#PWR0904")
 					(unit 1)
 				)
@@
 		(dnp no)
 		(fields_autoplaced yes)
-		(property "Reference" "R301"
+		(property "Reference" "R901"
 			(at 124.46 83.8199 0)
 			(effects
@@
 			(project "main"
 				(path "/f228839c-6576-40b2-ae70-679b7b460639/9647d80f-843f-45c0-950d-b04b6dbce3c2"
-					(reference "R301")
+					(reference "R901")
 					(unit 1)
 				)
@@
 		(dnp no)
 		(fields_autoplaced yes)
-		(property "Reference" "U301"
+		(property "Reference" "U901"
 			(at 145.6533 71.12 0)
 			(effects
@@
 			(project "main"
 				(path "/f228839c-6576-40b2-ae70-679b7b460639/9647d80f-843f-45c0-950d-b04b6dbce3c2"
-					(reference "U301")
+					(reference "U901")
 					(unit 1)
 				)

Commit message: update pcb
Connections:
- net +5V renamed +3V3
Changed lines of the file:
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@@
+	)
+	(symbol
+		(lib_id "power:+3V3")
+		(at 143.51 68.58 0)
+		(unit 1)
+		(exclude_from_sim no)
+		(in_bom yes)
+		(on_board yes)
+		(dnp no)
+		(fields_autoplaced yes)
+		(property "Reference" "#PWR0901"
+			(at 143.51 72.39 0)
+			(effects
+				(font
+					(size 1.27 1.27)
+				)
+				(hide yes)
+			)
+		)
+		(property "Value" "+3V3"
+			(at 143.51 63.5 0)
+			(effects
+				(font
+					(size 1.27 1.27)
+				)
+			)
+		)
+		(property "Footprint" ""
+			(at 143.51 68.58 0)
+			(effects
+				(font
+					(size 1.27 1.27)
+				)
+				(hide yes)
+			)
+		)
+		(property "Datasheet" ""
+			(at 143.51 68.58 0)
+			(effects
+				(font
+					(size 1.27 1.27)
+				)
+				(hide yes)
+			)
+		)
+		(property "Description" "Power symbol creates a global label with name \"+3V3\""
+			(at 143.51 68.58 0)
+			(effects
+				(font
+					(size 1.27 1.27)
+				)
+				(hide yes)
+			)
+		)
+		(pin "1"
+		)
+		(instances
+			(project ""
+				(path "/f228839c-6576-40b2-ae70-679b7b460639/9647d80f-843f-45c0-950d-b04b6dbce3c2"
+					(reference "#PWR0901")
+					(unit 1)
+				)
+			)
+		)
 	)
 	(symbol
@@
 	)
 	(symbol
-		(lib_id "power:+5V")
+		(lib_id "power:GND")
+		(at 176.53 88.9 0)
+		(unit 1)
+		(exclude_from_sim no)
+		(in_bom yes)
+		(on_board yes)
+		(dnp no)
+		(fields_autoplaced yes)
+		(property "Reference" "#PWR0904"
+			(at 176.53 95.25 0)
+			(effects
+				(font
+					(size 1.27 1.27)
+				)
+				(hide yes)
+			)
+		)
+		(property "Value" "GND"
+			(at 176.53 93.98 0)
+			(effects
+				(font
+					(size 1.27 1.27)
+				)
+			)
+		)
+		(property "Footprint" ""
+			(at 176.53 88.9 0)
+			(effects
+				(font
+					(size 1.27 1.27)
+				)
+				(hide yes)
+			)
+		)
+		(property "Datasheet" ""
+			(at 176.53 88.9 0)
+			(effects
+				(font
+					(size 1.27 1.27)
+				)
+				(hide yes)
+			)
+		)
+		(property "Description" "Power symbol creates a global label with name \"GND\" , ground"
+			(at 176.53 88.9 0)
+			(effects
+				(font
+					(size 1.27 1.27)
+				)
+				(hide yes)
+			)
+		)
+		(pin "1"
+		)
+		(instances
+			(project "main"
+				(path "/f228839c-6576-40b2-ae70-679b7b460639/9647d80f-843f-45c0-950d-b04b6dbce3c2"
+					(reference "#PWR0904")
+					(unit 1)
+				)
+			)
+		)
+	)
+	(symbol
+		(lib_id "power:+3V3")
 		(at 176.53 74.93 0)
 		(unit 1)
@@
 			)
 		)
-		(property "Value" "+5V"
+		(property "Value" "+3V3"
 			(at 176.53 69.85 0)
 			(effects
@@
 			)
 		)
-		(property "Description" "Power symbol creates a global label with name \"+5V\""
+		(property "Description" "Power symbol creates a global label with name \"+3V3\""
 			(at 176.53 74.93 0)
 			(effects
@@
 			)
 		)
-		(property "LCSC" ""
-			(at 176.53 74.93 0)
-			(effects
-				(font
-					(size 1.27 1.27)
-				)
-				(hide yes)
-			)
-		)
 		(pin "1"
 		)
@@
 					(unit 1)
 				)
-			)
-		)
-	)
-	(symbol
-		(lib_id "power:GND")
-		(at 176.53 88.9 0)
-		(unit 1)
-		(exclude_from_sim no)
-		(in_bom yes)
-		(on_board yes)
-		(dnp no)
-		(fields_autoplaced yes)
-		(property "Reference" "#PWR0904"
-			(at 176.53 95.25 0)
-			(effects
-				(font
-					(size 1.27 1.27)
-				)
-				(hide yes)
-			)
-		)
-		(property "Value" "GND"
-			(at 176.53 93.98 0)
-			(effects
-				(font
-					(size 1.27 1.27)
-				)
-			)
-		)
-		(property "Footprint" ""
-			(at 176.53 88.9 0)
-			(effects
-				(font
-					(size 1.27 1.27)
-				)
-				(hide yes)
-			)
-		)
-		(property "Datasheet" ""
-			(at 176.53 88.9 0)
-			(effects
-				(font
-					(size 1.27 1.27)
-				)
-				(hide yes)
-			)
-		)
-		(property "Description" "Power symbol creates a global label with name \"GND\" , ground"
-			(at 176.53 88.9 0)
-			(effects
-				(font
-					(size 1.27 1.27)
-				)
-				(hide yes)
-			)
-		)
-		(pin "1"
-		)
-		(instances
-			(project "main"
-				(path "/f228839c-6576-40b2-ae70-679b7b460639/9647d80f-843f-45c0-950d-b04b6dbce3c2"
-					(reference "#PWR0904")
-					(unit 1)
-				)
-			)
-		)
-	)
-	(symbol
-		(lib_id "power:+5V")
-		(at 143.51 68.58 0)
-		(unit 1)
-		(exclude_from_sim no)
-		(in_bom yes)
-		(on_board yes)
-		(dnp no)
-		(fields_autoplaced yes)
-		(property "Reference" "#PWR0901"
-			(at 143.51 72.39 0)
-			(effects
-				(font
-					(size 1.27 1.27)
-				)
-				(hide yes)
-			)
-		)
-		(property "Value" "+5V"
-			(at 143.51 63.5 0)
-			(effects
-				(font
-					(size 1.27 1.27)
-				)
-			)
-		)
-		(property "Footprint" ""
-			(at 143.51 68.58 0)
-			(effects
-				(font
-					(size 1.27 1.27)
-				)
-				(hide yes)
-			)
-		)
-		(property "Datasheet" ""
-			(at 143.51 68.58 0)
-			(effects
-				(font
-					(size 1.27 1.27)
-				)
-				(hide yes)
-			)
-		)
-		(property "Description" "Power symbol creates a global label with name \"+5V\""
-			(at 143.51 68.58 0)
-			(effects
-				(font
-					(size 1.27 1.27)
-				)
-				(hide yes)
-			)
-		)
-		(property "LCSC" ""
-			(at 143.51 68.58 0)
-			(effects
-				(font
-					(size 1.27 1.27)
-				)
-				(hide yes)
-			)
-		)
-		(pin "1"
-		)
-		(instances
-			(project "main"
-				(path "/f228839c-6576-40b2-ae70-679b7b460639/9647d80f-843f-45c0-950d-b04b6dbce3c2"
-					(reference "#PWR0901")
-					(unit 1)
-				)
