File: sw_port.kicad_sch (KiCad schematic)
At the start: 1 part, among them J1101 Conn_02x05_Odd_Even

Commit message: Update USB-C and USB-Hub Schematics with New Titles and Reference Changes
- Changed title from "DebugBoard" to "USB-C" in usb_c.kicad_sch.
- Changed title from "DebugBoard" to "USB-Hub" in usb_hub.kicad_sch.
- Updated multiple component references in usb_c.kicad_sch to new identifiers (#PWR0301 to #PWR0312, D301, U301, etc.).
- Updated component reference from "R103" to "R501" in usb_hub.kicad_sch.
Other:
- title: DebugBoard -> SW Port
Changed lines of the file:
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@@
 	(paper "A4")
 	(title_block
-		(title "DebugBoard")
+		(title "SW Port")
 		(rev "<<HASH>>")
 		(company "Amateurfunkclub für Remote Stationen")
@@
 		(dnp no)
 		(fields_autoplaced yes)
-		(property "Reference" "#PWR01102"
+		(property "Reference" "#PWR01101"
 			(at 144.78 97.79 0)
 			(effects
@@
 			(project "main"
 				(path "/f228839c-6576-40b2-ae70-679b7b460639/2986b648-d6e4-4f37-95a0-c0a0bf4ce6d9/7fb85a85-298d-489a-83e9-b51a73cb28d0"
-					(reference "#PWR01102")
+					(reference "#PWR01101")
 					(unit 1)
 				)
 				(path "/f228839c-6576-40b2-ae70-679b7b460639/4f8158b0-0961-44de-9899-c669fc1a50b4/4de6f778-d6ef-4181-8ca5-1bc42ed36179"
-					(reference "#PWR01202")
+					(reference "#PWR01201")
 					(unit 1)
 				)
@@
 		(dnp no)
 		(fields_autoplaced yes)
-		(property "Reference" "#PWR01101"
+		(property "Reference" "#PWR01102"
 			(at 163.83 97.79 0)
 			(effects
@@
 			(project ""
 				(path "/f228839c-6576-40b2-ae70-679b7b460639/2986b648-d6e4-4f37-95a0-c0a0bf4ce6d9/7fb85a85-298d-489a-83e9-b51a73cb28d0"
-					(reference "#PWR01101")
+					(reference "#PWR01102")
 					(unit 1)
 				)
 				(path "/f228839c-6576-40b2-ae70-679b7b460639/4f8158b0-0961-44de-9899-c669fc1a50b4/4de6f778-d6ef-4181-8ca5-1bc42ed36179"
-					(reference "#PWR01201")
-					(unit 1)
-				)
+					(reference "#PWR01202")
+					(unit 1)
+				)

Commit message: update pcb
Parts:
- J1101: footprint (none) -> Connector_IDC:IDC-Header_2x05_P2.54mm_Vertical
Changed lines of the file:
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@@
 			)
 		)
-		(property "Footprint" ""
+		(property "Footprint" "Connector_IDC:IDC-Header_2x05_P2.54mm_Vertical"
 			(at 152.4 83.82 0)
 			(effects
@@
 			(at 152.4 83.82 0)
 			(effects
+				(font
+					(size 1.27 1.27)
+				)
+				(hide yes)
+			)
+		)
+		(property "LCSC" ""
+			(at 152.4 83.82 0)
+			(effects
