File: ui.kicad_sch (KiCad schematic)
At the start: 0 parts

Commit message: Update USB-C and USB-Hub Schematics with New Titles and Reference Changes
- Changed title from "DebugBoard" to "USB-C" in usb_c.kicad_sch.
- Changed title from "DebugBoard" to "USB-Hub" in usb_hub.kicad_sch.
- Updated multiple component references in usb_c.kicad_sch to new identifiers (#PWR0301 to #PWR0312, D301, U301, etc.).
- Updated component reference from "R103" to "R501" in usb_hub.kicad_sch.
Parts:
- added Brd701: SSD1306, PRJ:128x64OLED, symbol SSD1306:SSD1306
- added SW701, SW702, SW703: SW_Push, symbol Switch:SW_Push
Connections:
- new net +3V3: Brd701.2 (VCC)
- new net BUTTON_DOWN: SW703.1
- new net BUTTON_OK: SW702.1
- new net BUTTON_UP: SW701.1
- new net GND: Brd701.1 (GND), SW701.2, SW702.2, SW703.2
- new net I2C_SCL: Brd701.3 (SCL)
- new net I2C_SDA: Brd701.4 (SDA)
Other:
- title: DebugBoard -> Display & UI

Commit message: update pcb
Parts:
- SW701, SW702, SW703: footprint (none) -> Button_Switch_THT:SW_PUSH_6mm
Changed lines of the file:
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@@
 			)
 		)
-		(property "Footprint" ""
+		(property "Footprint" "Button_Switch_THT:SW_PUSH_6mm"
 			(at 107.95 86.36 0)
 			(effects
@@
 			)
 		)
+		(property "LCSC" ""
+			(at 107.95 91.44 0)
+			(effects
+				(font
+					(size 1.27 1.27)
+				)
+				(hide yes)
+			)
+		)
 		(pin "2"
 		)
@@
 			)
 		)
-		(property "Footprint" ""
+		(property "Footprint" "Button_Switch_THT:SW_PUSH_6mm"
 			(at 107.95 55.88 0)
 			(effects
@@
 			)
 		)
+		(property "LCSC" ""
+			(at 107.95 60.96 0)
+			(effects
+				(font
+					(size 1.27 1.27)
+				)
+				(hide yes)
+			)
+		)
 		(pin "2"
 		)
@@
 			)
 		)
-		(property "Footprint" ""
+		(property "Footprint" "Button_Switch_THT:SW_PUSH_6mm"
 			(at 107.95 71.12 0)
 			(effects
@@
 			(at 107.95 76.2 0)
 			(effects
+				(font
+					(size 1.27 1.27)
+				)
+				(hide yes)
+			)
+		)
+		(property "LCSC" ""
+			(at 107.95 76.2 0)
+			(effects
